File: Pcb/room.kicad_pcb (KiCad board)
At the start: 4 copper layers, 79 x 100 mm, 38 parts, among them J1 USB_C_Receptacle_USB2.0_14P, J2 Screw_Terminal_01x10, J3 BOOT, J4 Screw_Terminal_01x03, K1 D1, K2 D2, K3 D3, K4 D4, Q1 BC547, Q2 BC547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

Commit message: Mostly done
Parts:
- removed J2: Screw_Terminal_01x10, TerminalBlock:TerminalBlock_Xinya_XY308-2.54-10P_1x10_P2.54mm_Horizontal
- removed J4: Screw_Terminal_01x03, TerminalBlock:TerminalBlock_Xinya_XY308-2.54-3P_1x03_P2.54mm_Horizontal
- added J5: Screw_Terminal_01x06, TerminalBlock:TerminalBlock_bornier-6_P5.08mm, F.Cu at (155.0, 79.2)
- added REF**: MountingHole_2.7mm_M2.5, MountingHole:MountingHole_2.7mm_M2.5, F.Cu at (226.0, 147.0)
- added REF**: MountingHole_2.7mm_M2.5, MountingHole:MountingHole_2.7mm_M2.5, F.Cu at (226.0, 53.0)
- added REF**: MountingHole_2.7mm_M2.5, MountingHole:MountingHole_2.7mm_M2.5, F.Cu at (153.0, 147.0)
- added REF**: ESD-Logo_33x30mm_SilkScreen, Symbol:ESD-Logo_33x30mm_SilkScreen, B.Cu at (189.5, 69.5)
- added kibuzzard-69B63945: G***, kibuzzard-69B63945, F.Cu at (165.2, 53.5)
- added kibuzzard-69B63945: G***, kibuzzard-69B63945, B.Cu at (165.2, 53.5)
- added kibuzzard-69B63969: G***, kibuzzard-69B63969, F.Cu at (171.0, 115.0)
- added kibuzzard-69B63969: G***, kibuzzard-69B63969, B.Cu at (171.0, 115.0)
- moved R3 11.2 mm to (213.0, 147.0), turned to -90 degrees
- moved C7 8.12 mm to (225.1, 67.0)
- moved PS1 8.12 mm to (177.1, 63.1)
- moved C6 7.33 mm to (227.3, 67.0)
- moved C5 4.00 mm to (218.0, 145.8)
- moved D7 4.00 mm to (164.0, 129.0)
- moved SW1 2.02 mm to (220.0, 143.2)
Routing:
- net L: track 481.1 -> 388.8 mm
- net N: track 64.0 -> 23.4 mm
- net /D4: track 95.8 -> 83.9 mm
- net 5V: track 36.4 -> 45.0 mm, vias 0 -> 1
- net /EN: track 18.8 -> 11.2 mm
- net /D3: track 75.0 -> 70.1 mm
- net Net-(D5-K): track 24.0 -> 20.0 mm
- net /D2: track 51.8 -> 48.1 mm
- net GND: track 41.4 -> 38.7 mm, vias 10 -> 9
- net +3V3: track 15.1 -> 13.8 mm
- net /D1: track 33.8 -> 33.1 mm
Other:
- board text added: "_____________________________________________________________________"
