File: Pcb/room.kicad_pcb (KiCad board)
At the start: 4 copper layers, 79 x 100 mm, 45 parts, among them J1 USB_C_Receptacle_USB2.0_14P, J3 BOOT, J5 Screw_Terminal_01x06, K1 D1, K2 D2, K3 D3, K4 D4, Q1 BC547, Q2 BC547, Q3 BC547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

Commit message: Final update for pcb
Parts:
- removed C5: .1uF, Capacitor_SMD:C_0603_1608Metric_Pad1.08x0.95mm_HandSolder
- removed J3: BOOT, Connector_PinHeader_2.54mm:PinHeader_1x02_P2.54mm_Vertical
- removed the REF** at (226.0, 147.0)
- removed the REF** at (226.0, 53.0)
- removed the REF** at (153.0, 147.0)
- removed the REF** at (189.5, 69.5)
- removed SW1: SW_Push, Button_Switch_SMD:SW_Push_SPST_NO_Alps_SKRK
- removed U1: ESP32-C3-WROOM-02, RF_Module:ESP32-C3-WROOM-02
- removed the kibuzzard-69B63945 at (165.2, 53.5)
- removed the kibuzzard-69B63969 at (171.0, 115.0)
- added DL1: LED, LED_SMD:LED_0805_2012Metric_Pad1.15x1.40mm_HandSolder, F.Cu at (200.0, 128.5)
- added DL2: LED, LED_SMD:LED_0805_2012Metric_Pad1.15x1.40mm_HandSolder, F.Cu at (185.5, 128.5)
- added DL3: LED, LED_SMD:LED_0805_2012Metric_Pad1.15x1.40mm_HandSolder, F.Cu at (197.0, 125.0)
- added DL4: LED, LED_SMD:LED_0805_2012Metric_Pad1.15x1.40mm_HandSolder, F.Cu at (227.0, 71.5)
- added DL5: LED, LED_SMD:LED_0805_2012Metric_Pad1.15x1.40mm_HandSolder, F.Cu at (184.0, 143.0)
- added G***: LOGO, LOGO, B.Cu at (198.0, 124.0)
- added H1: MountingHole, MountingHole:MountingHole_2.5mm, F.Cu at (154.0, 142.5)
- added H2: MountingHole, MountingHole:MountingHole_2.5mm, F.Cu at (202.0, 142.5)
- added H3: MountingHole, MountingHole:MountingHole_2.5mm, F.Cu at (154.0, 115.0)
- added H4: MountingHole, MountingHole:MountingHole_2.5mm, F.Cu at (225.5, 115.0)
- added H5: MountingHole, MountingHole:MountingHole_2.5mm, F.Cu at (202.0, 115.0)
- added H6: MountingHole, MountingHole:MountingHole_2.5mm, F.Cu at (225.5, 85.0)
- added J2: Conn_01x05_Pin, Connector_PinHeader_2.54mm:PinHeader_1x05_P2.54mm_Vertical, F.Cu at (215.9, 126.0)
- added R10: 330, PCM_SparkFun-Resistor:R_0603_1608Metric, F.Cu at (226.3, 75.0)
- added R11: 330, PCM_SparkFun-Resistor:R_0603_1608Metric, F.Cu at (183.5, 145.0)
- added REF**: ESD-Logo_6.6x6mm_SilkScreen, Symbol:ESD-Logo_6.6x6mm_SilkScreen, F.Cu at (158.0, 127.5)
- added REF**: KiCad-Logo2_5mm_SilkScreen, Symbol:KiCad-Logo2_5mm_SilkScreen, F.Cu at (158.0, 134.5)
- added REF**: ESD-Logo_6.6x6mm_SilkScreen, Symbol:ESD-Logo_6.6x6mm_SilkScreen, F.Cu at (157.8, 85.5)
- added REF**: UKCA-Logo_6x6mm_SilkScreen, Symbol:UKCA-Logo_6x6mm_SilkScreen, F.Cu at (165.5, 145.5)
- added U3: XIAO-ESP32-S3-DIP, Seeed Studio XIAO Series Library:XIAO-ESP32S3-DIP, F.Cu at (216.4, 139.4)
- added kibuzzard-69C64D69: G***, kibuzzard-69C64D69, F.Cu at (193.0, 64.0)
- R3, R4, R5: value 10K -> 220
- moved R4 35.5 mm to (181.5, 128.5)
- moved kibuzzard-69B63969 27.2 mm to (193.0, 131.0)
- moved R5 24.2 mm to (200.5, 125.0)
- moved R3 20.7 mm to (203.8, 128.5), turned to 180 degrees
- moved D5 1.75 mm to (167.5, 138.0)
- moved D7 1.00 mm to (165.0, 129.0)
Connections:
- R3 pad 1: +3V3 -> GND
- R3 pad 2: /EN -> Net-(DL1-A)
- R4 pad 1: /S8 -> GND
- R4 pad 2: +3V3 -> Net-(DL2-A)
- R5 pad 1: /S2 -> GND
- R5 pad 2: +3V3 -> Net-(DL3-A)
Routing:
- net /Led2: track 0.00 -> 26.3 mm, vias 0 -> 1
- net /D-: track 23.4 -> 2.44 mm
- net /D+: track 23.4 -> 2.44 mm
- net /DT1: track 58.3 -> 74.6 mm, vias 0 -> 1
- net /Led1: track 0.00 -> 14.6 mm
- net /DT2: track 40.7 -> 54.8 mm
- net /sda: track 0.00 -> 13.3 mm
- net /rx: track 0.00 -> 13.0 mm, vias 0 -> 2
- net /scl: track 0.00 -> 12.4 mm
- net /sck: track 0.00 -> 12.1 mm, vias 0 -> 1
- net +3V3: track 13.8 -> 2.56 mm, vias 4 -> 0
- net /EN: track 11.2 -> 0.00 mm
- net /DT3: track 28.6 -> 37.6 mm
- net GND: track 38.7 -> 46.8 mm, vias 9 -> 8
- net /tx: track 0.00 -> 7.37 mm
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Other:
- board text added: "BC547"
- board text added: "Contact me@souptik.me"
- board text added: "JLCJLCJLC"
- board text added: "JLCJLCJLCJLC"
- board text added: "Made by SoupIndustries"
- board text removed: "_____________________________________________________________________"
