File: Pcb/room.kicad_sch (KiCad schematic)
At the start: 38 parts, among them J1 USB_C_Receptacle_USB2.0_14P, J2 Screw_Terminal_01x10, J3 BOOT, J4 Screw_Terminal_01x03, K1 D1, K2 D2, K3 D3, K4 D4, Q1 BC547, Q2 BC547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

Commit message: Mostly done
Parts:
- removed J2: Screw_Terminal_01x10, TerminalBlock:TerminalBlock_Xinya_XY308-2.54-10P_1x10_P2.54mm_Horizontal, symbol Connector:Screw_Terminal_01x10
- removed J4: Screw_Terminal_01x03, TerminalBlock:TerminalBlock_Xinya_XY308-2.54-3P_1x03_P2.54mm_Horizontal, symbol Connector:Screw_Terminal_01x03
- added J5: Screw_Terminal_01x06, TerminalBlock:TerminalBlock_bornier-6_P5.08mm, symbol Connector:Screw_Terminal_01x06
Connections:
- net D1: now also J5.3 (Pin_3)
- net D2: now also J5.4 (Pin_4)
- net D3: now also J5.5 (Pin_5)
- net D4: now also J5.6 (Pin_6)
- net L: now also J5.1 (Pin_1)
- net N: now also J5.2 (Pin_2)

Commit message: Final update for pcb
Parts:
- removed C5: .1uF, Capacitor_SMD:C_0603_1608Metric_Pad1.08x0.95mm_HandSolder, symbol Device:C
- removed J3: BOOT, Connector_PinHeader_2.54mm:PinHeader_1x02_P2.54mm_Vertical, symbol Connector:Conn_01x02_Pin
- removed SW1: SW_Push, Button_Switch_SMD:SW_Push_SPST_NO_Alps_SKRK, symbol Switch:SW_Push
- removed U1: ESP32-C3-WROOM-02, RF_Module:ESP32-C3-WROOM-02, symbol RF_Module:ESP32-C3-WROOM-02
- added DL1, DL2, DL3, DL4, DL5: LED, LED_SMD:LED_0805_2012Metric_Pad1.15x1.40mm_HandSolder, symbol PCM_SparkFun-LED:LED
- added H1, H2, H3, H4, H5, H6: MountingHole, MountingHole:MountingHole_2.5mm, symbol Mechanical:MountingHole
- added J2: Conn_01x05_Pin, Connector_PinHeader_2.54mm:PinHeader_1x05_P2.54mm_Vertical, symbol Connector:Conn_01x05_Pin
- added R10, R11: 330, PCM_SparkFun-Resistor:R_0603_1608Metric, symbol Device:R
- added U3: XIAO-ESP32-S3-DIP, Seeed Studio XIAO Series Library:XIAO-ESP32S3-DIP, symbol Seeed_Studio_XIAO_Series:XIAO-ESP32-S3-DIP
- R3, R4, R5: value 10K -> 220
Connections:
- net S2 is gone; now on net GND: R5.1
- net S8 is gone; now on net GND: R4.1
- net +3V3: now also DL3.1 (K), U3.12 (VCC_3V3); no longer R3.1, R4.2, R5.2
- net 5V: now also DL4.1 (K)
- net DT1: now also U3.1 (GPIO1/D0/A0)
- net DT2: now also U3.2 (GPIO2/DA/A1)
- net DT3: now also U3.3 (GPIO3/D2/A2)
- net DT4: now also U3.4 (GPIO4/D3/A3)
- net GND: now also R3.1, R10.1, R11.1, U3.13 (GND)
- net VBUS: now also DL5.1 (K)
- net EN: no longer names the net of R3.2
- net EN: now also DL1.2 (A)
- new net: DL2.2 (A), R4.2
- new net: DL4.2 (A), R10.2
- new net: DL3.2 (A), R5.2
- new net: DL5.2 (A), R11.2
- new net Led1: DL1.1 (K), U3.11 (GPIO9/D10/A10/MOSI)
- new net Led2: DL2.1 (K), U3.10 (GPIO8/D9/A9/MISO)
- new net rx: J2.2 (Pin_2), U3.8 (U0RXD/D7/RX)
- new net sck: J2.1 (Pin_1), U3.9 (GPIO7/D8/A8/SCK)
- new net scl: J2.4 (Pin_4), U3.6 (GPIO9/D5/I2C_SCL)
- new net sda: J2.5 (Pin_5), U3.5 (GPIO5/D4/I2C_SDA)
- new net tx: J2.3 (Pin_3), U3.7 (U0TXD/D6/TX)
